Commit message: removed camera and added odometry filter.

File: mode_3/mode_3_ws/src/bondk/bondk_desc/urdf/bondk.xacro (robot description, xacro)
@@ -1,6 +1,6 @@
 <?xml version='1.0'?>
 <robot name="bondk" xmlns:xacro="http://www.ros.org/wiki/xacro">
-  <xacro:property name="cameraSize" value="0.05"/>
-  <xacro:property name="cameraMass" value="0.1"/>
+  <!-- <xacro:property name="cameraSize" value="0.05"/>
+  <xacro:property name="cameraMass" value="0.1"/> -->
   <xacro:include filename="$(find bondk_desc)/urdf/materials.xacro"/>
   <xacro:include filename="$(find bondk_desc)/urdf/bondk.gazebo"/>
@@ -128,5 +128,5 @@
     <child link="chassis"/>
   </joint>
-  <!-- Camera -->
+  <!-- Camera
   <link name="camera_link">
     <collision>
@@ -155,5 +155,5 @@
     <parent link="chassis"/>
     <child link="camera_link"/>
-  </joint>
+  </joint> -->
    <!-- Hokuyo Laser -->
   <link name="hokuyo_link">

Commit message: 2d mapping maybe done.

File: mode_3/mode_3_ws/src/bondk/bondk_desc/urdf/bondk.xacro (robot description, xacro)
@@ -178,5 +178,5 @@
   <joint name="hokuyo_joint" type="fixed">
     <axis xyz="0 1 0" />
-    <origin xyz="0.15 0 0.1" rpy="0 0 0"/>
+    <origin xyz="0.15 0 0.15" rpy="0 0 0"/>
     <parent link="chassis"/>
     <child link="hokuyo_link"/>
